File: kicad/handheld.kicad_pcb (KiCad board)
At the start: 2 copper layers, 19 parts, among them J1 CONN_02X03, Q1 BSS138, SW1 LEFT, SW2 RIGHT, SW3 POWER, U1 ATTINY88-AU, U2 4027

Commit message: dflsj
Parts:
- removed C1: 33n, Capacitors_SMD:C_0805_HandSoldering
- removed LEFT_R1, R1, R2, R3, R4, R5, RIGHT_R1: 2k, Resistors_SMD:R_0805_HandSoldering
- removed R10, R11: 100k, Resistors_SMD:R_0805_HandSoldering
- removed SW1: LEFT, Buttons_Switches_SMD:SW_SPST_EVPBF
- removed SW2: RIGHT, Buttons_Switches_SMD:SW_SPST_EVPBF
- added 100k: 100k, Resistors_SMD:R_0805, B.Cu at (117.5, 97.8)
- added 100k: 100k, Resistors_SMD:R_0805, B.Cu at (120.1, 97.8)
- added 100k: 100k, Resistors_SMD:R_0805, B.Cu at (134.6, 102.1)
- added 100k: 100k, Resistors_SMD:R_0805, B.Cu at (119.4, 102.1)
- added 2k: 2k, Resistors_SMD:R_0805, F.Cu at (117.0, 85.9)
- added 2k: 2k, Resistors_SMD:R_0805, F.Cu at (120.0, 85.9)
- added 2k: 2k, Resistors_SMD:R_0805, F.Cu at (114.6, 89.3)
- added 2k: 2k, Resistors_SMD:R_0805, F.Cu at (113.9, 85.9)
- added 2k: 2k, Resistors_SMD:R_0805, F.Cu at (119.4, 89.3)
- added CAP: 33n, Capacitors_SMD:C_0805, F.Cu at (110.7, 93.7)
- added G***: LOGO, kicad_bart:logo, F.Cu at (119.1, 92.8)
- added LEFT: LEFT, kicad_bart:SW_PANASONIC, F.Cu at (114.3, 99.1)
- added RIGHT: RIGHT, kicad_bart:SW_PANASONIC, F.Cu at (139.7, 99.1)
- BT1: footprint Resistors_SMD:R_2816 -> kicad_bart:BatteryHolder_1220
- J1: footprint Pin_Headers:Pin_Header_Straight_2x03 -> kicad_bart:Pin_Header_2x3_SMD
- Q1: moved to F.Cu
- S1: footprint Displays_7-Segment:MAN3640A -> kicad_bart:2x7_dot_matrix
- SW3: footprint Buttons_Switches_SMD:SW_SPST_EVPBF -> kicad_bart:SW_OMRON_SMALL
- moved Q1 33.4 mm to (114.8, 93.0)
- moved U2 31.3 mm to (114.6, 88.9)
- moved BT1 28.8 mm to (139.4, 93.3), turned to 270 degrees
- moved J1 26.7 mm to (113.4, 96.5), turned to 180 degrees
- moved SW3 3.99 mm to (110.4, 86.6), turned to 90 degrees
- moved U1 1.61 mm to (139.7, 88.9), turned to 90 degrees
- moved S1 0.83 mm to (127.0, 93.3), turned to 270 degrees
Connections:
- BT1 pad 2: Net-(BT1-Pad2) -> GND
- J1 pad 6: VCC -> Net-(J1-Pad6)
- Q1 pad 2: GND -> Net-(J1-Pad6)
- Q1 pad 3: Net-(BT1-Pad2) -> VCC
- SW3 pad 1: Net-(SW3-Pad1) -> Net-(C1-Pad1)
- SW3 pad 2: Net-(SW3-Pad2) -> VCC
- U1 pad 1: Net-(U1-Pad1) -> Net-(S1-Pad7)
- U1 pad 18: VCC -> Net-(J1-Pad6)
- U1 pad 22: Net-(R2-Pad2) (its old number) -> Net-(S1-Pad3)
- U1 pad 23: Net-(S1-Pad3) -> Net-(S1-Pad2)
- U1 pad 24: Net-(S1-Pad4) -> Net-(R4-Pad2)
- U1 pad 27: Net-(S1-Pad9) -> Net-(S1-Pad12)
- U1 pad 28: Net-(U1-Pad28) -> Net-(S1-Pad11)
- U1 pad 30: Net-(U1-Pad30) -> Net-(S1-Pad10)
- U1 pad 31: Net-(U1-Pad31) -> Net-(S1-Pad4)
- U1 pad 32: Net-(U1-Pad32) -> Net-(S1-Pad9)
- U1 pad 4: VCC -> Net-(J1-Pad6)
- U1 pad 7: Net-(S1-Pad2) -> Net-(U1-Pad7)
- U1 pad 8: Net-(S1-Pad12) -> Net-(U1-Pad8)
- U2 pad 10: Net-(U2-Pad10) -> GND
- U2 pad 11: Net-(U2-Pad10) -> GND
- U2 pad 12: Net-(U2-Pad10) -> GND
- U2 pad 13: Net-(U2-Pad10) -> GND
- U2 pad 9: Net-(U2-Pad10) -> GND
Routing:
- net Net-(J1-Pad6): track 0.00 -> 61.4 mm, vias 0 -> 1
- net Net-(J1-Pad4): track 0.00 -> 52.7 mm, vias 0 -> 1
- net Net-(SW1-Pad1): track 0.00 -> 43.6 mm, vias 0 -> 2
- net Net-(R3-Pad2): track 0.00 -> 41.7 mm
- net Net-(J1-Pad5): track 0.00 -> 41.7 mm, vias 0 -> 1
- net Net-(J1-Pad2): track 0.00 -> 40.2 mm, vias 0 -> 1
- net Net-(J1-Pad3): track 0.00 -> 39.7 mm, vias 0 -> 1
- net Net-(R5-Pad2): track 0.00 -> 35.1 mm
- net Net-(R3-Pad1): track 0.00 -> 26.8 mm
- net Net-(R4-Pad2): track 0.00 -> 24.2 mm
- net Net-(C1-Pad1): track 0.00 -> 22.0 mm, vias 0 -> 1
- net Net-(R1-Pad2): track 0.00 -> 20.3 mm
- net Net-(S1-Pad3): track 0.00 -> 19.4 mm, vias 0 -> 2
- net Net-(S1-Pad7): track 0.00 -> 18.7 mm
- net Net-(S1-Pad2): track 0.00 -> 18.3 mm, vias 0 -> 2
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- added copper zone on B.Cu, net GND
- added copper zone on F.Cu, net VCC
Other:
- board outline added: 38.1 x 21.6 mm
- net class Default: clearance 0.2 -> 0.1; trace_width 0.25 -> 0.1; via_dia 0.6 -> 0.45; via_drill 0.4 -> 0.2
- rule trace_clearance: 0.2 -> 0.1
- rule trace_min: 0.2 -> 0.1
- rule via_min_drill: 0.3 -> 0.2
- rule via_min_size: 0.4 -> 0.45
- board text added: "2017"
