File: kicad/handheld.sch (KiCad schematic (older format))
At the start: 19 parts, among them J1 CONN_02X03, Q1 BSS138, SW1 LEFT, SW2 RIGHT, SW3 POWER, U1 ATTINY88-AU, U2 4027

Commit message: dflsj
Parts:
- C1: footprint Capacitors_SMD:C_0805_HandSoldering -> Capacitors_SMD:C_0805
- J1: footprint Pin_Headers:Pin_Header_Straight_2x03 -> kicad_bart:Pin_Header_2x3_SMD
- LEFT_R1, RIGHT_R1: value 2k -> 100k; footprint Resistors_SMD:R_0805_HandSoldering -> Resistors_SMD:R_0805
- Q1: symbol BSS138 -> BSS138-RESCUE-handheld
- R1, R10, R11, R2, R3, R4, R5: footprint Resistors_SMD:R_0805_HandSoldering -> Resistors_SMD:R_0805
- S1: footprint Displays_7-Segment:MAN3640A -> kicad_bart:2x7_dot_matrix
- SW1, SW2: footprint Buttons_Switches_SMD:SW_SPST_EVPBF -> kicad_bart:SW_PANASONIC; symbol Rotary_Encoder_Switch -> Switch
- SW3: footprint Buttons_Switches_SMD:SW_SPST_EVPBF -> kicad_bart:SW_OMRON_SMALL; symbol Rotary_Encoder_Switch -> Switch
Connections:
- net GND: now also BT1.2 (-), U2.10 (J), U2.11 (K), U2.12 (Cd), U2.13 (Cp), U2.9 (Sd); no longer Q1.2 (S)
- net VCC: now also Q1.3 (D), SW3.2; no longer J1.6 (P6), SW3.5, U1.18 (AVCC), U1.4 (VCC)
- net at U1.1 ((PCINT19/INT1)PD3): now also S1.7 (DECIMAL)
- net at U1.10 ((PCINT22/AIN0)PD6): now also SW2.1; no longer SW1.4
- net at U1.11 ((PCINT23/AIN1)PD7): now also SW1.1; no longer SW2.4
- net at U1.12 ((PCINT0/CLKO/ICP1)PB0): no longer R5.2
- net at U1.19 ((PCINT24/ADC6)PA0): no longer R1.2
- net at U1.2 ((PCINT20/T0)PD4): now also R5.2
- net at U1.22 ((PCINT25/ADC7)PA1): now also S1.3 (ROW3); no longer R2.2
- net at U1.23 ((PCINT8/ADC0)PC0): now also S1.2 (ROW1); no longer S1.3 (ROW3)
- net at U1.24 ((PCINT9/ADC1)PC1): now also R4.2; no longer S1.4 (ROW4)
- net at U1.25 ((PCINT10/ADC2)PC2): now also R1.2; no longer S1.11 (ROW5)
- net at U1.26 ((PCINT11/ADC3)PC3): now also R2.2; no longer S1.10 (ROW6)
- net at U1.27 ((PCINT12/SDA/ADC4)PC4): now also S1.12 (ROW2); no longer S1.9 (ROW7)
- net at U1.28 ((PCINT13/SCL/ADC5)PC5): now also S1.11 (ROW5)
- net at U1.30 ((PCINT16)PD0): now also S1.10 (ROW6)
- net at U1.31 ((PCINT17)PD1): now also S1.4 (ROW4)
- net at U1.32 ((PCINT18/INT0)PD2): now also S1.9 (ROW7)
- net at U1.6 ((PCINT27)PA3): no longer R4.2
- net at U1.7 ((PCINT6/CLKI)PB6): no longer S1.2 (ROW1)
- net at U1.8 ((PCINT7)PB7): no longer S1.12 (ROW2)
- net at C1.1, R10.1, U2.3 (Cp): now also SW3.1; no longer SW3.4
- net at S1.13C (COL5): now also R2.1; no longer R5.1
- net at S1.14C (COL4): now also R1.1; no longer R4.1
- net at S1.1C (COL2): now also R4.1; no longer R2.1
- net at S1.5C (COL1): now also R5.1; no longer R1.1
- net at SW2.2: now also RIGHT_R1.1
- net at SW1.2: now also LEFT_R1.1
- new net: J1.6 (P6), Q1.2 (S), U1.18 (AVCC), U1.4 (VCC)
- no-connect marks 24 -> 12
Other:
- moved on the sheet: Q1

Commit message: Working scoring and horizontal scrolling.
Parts:
- LEFT_R1, RIGHT_R1: value 100k -> 2k
- R1, R2, R3, R4, R5: value 2k -> 20
Changed lines of the file:
@@
 P 5400 5300
 F 0 "RIGHT_R1" V 5480 5300 50  0000 C CNN
-F 1 "100k" V 5400 5300 50  0000 C CNN
+F 1 "2k" V 5400 5300 50  0000 C CNN
 F 2 "Resistors_SMD:R_0805" V 5330 5300 50  0001 C CNN
 F 3 "" H 5400 5300 50  0001 C CNN
@@
 P 5400 4350
 F 0 "LEFT_R1" V 5480 4350 50  0000 C CNN
-F 1 "100k" V 5400 4350 50  0000 C CNN
+F 1 "2k" V 5400 4350 50  0000 C CNN
 F 2 "Resistors_SMD:R_0805" V 5330 4350 50  0001 C CNN
 F 3 "" H 5400 4350 50  0001 C CNN
@@
 P 5650 1550
 F 0 "R1" V 5730 1550 50  0000 C CNN
-F 1 "2k" V 5650 1550 50  0000 C CNN
+F 1 "20" V 5650 1550 50  0000 C CNN
 F 2 "Resistors_SMD:R_0805" V 5580 1550 50  0001 C CNN
 F 3 "" H 5650 1550 50  0001 C CNN
@@
 P 5650 1700
 F 0 "R2" V 5730 1700 50  0000 C CNN
-F 1 "2k" V 5650 1700 50  0000 C CNN
+F 1 "20" V 5650 1700 50  0000 C CNN
 F 2 "Resistors_SMD:R_0805" V 5580 1700 50  0001 C CNN
 F 3 "" H 5650 1700 50  0001 C CNN
@@
 P 5650 1850
 F 0 "R3" V 5730 1850 50  0000 C CNN
-F 1 "2k" V 5650 1850 50  0000 C CNN
+F 1 "20" V 5650 1850 50  0000 C CNN
 F 2 "Resistors_SMD:R_0805" V 5580 1850 50  0001 C CNN
 F 3 "" H 5650 1850 50  0001 C CNN
@@
 P 5650 2000
 F 0 "R4" V 5730 2000 50  0000 C CNN
-F 1 "2k" V 5650 2000 50  0000 C CNN
+F 1 "20" V 5650 2000 50  0000 C CNN
 F 2 "Resistors_SMD:R_0805" V 5580 2000 50  0001 C CNN
 F 3 "" H 5650 2000 50  0001 C CNN
@@
 P 5650 2150
 F 0 "R5" V 5730 2150 50  0000 C CNN
-F 1 "2k" V 5650 2150 50  0000 C CNN
+F 1 "20" V 5650 2150 50  0000 C CNN
 F 2 "Resistors_SMD:R_0805" V 5580 2150 50  0001 C CNN
 F 3 "" H 5650 2150 50  0001 C CNN
