File: kicad/pcb.kicad_pcb (KiCad board)
At the start: 2 copper layers, 11 parts, among them J0 Conn_01x04, SW0 ON_OFF, SW4 RIGHT, SW7 LEFT, U0 STM32L031x4/6

Commit message: Getting there.
Parts:
- added C0: 100nF, Capacitors_SMD:C_0805_HandSoldering, B.Cu at (117.5, 62.6)
- J0: footprint Connect:bornier4 -> Pin_Headers:Pin_Header_Straight_1x04
- R0: moved to B.Cu
- moved J0 32.8 mm to (126.6, 63.1), turned to 0 degrees
- moved R0 29.1 mm to (110.6, 77.3), turned to 90 degrees
- moved R7 14.2 mm to (111.4, 62.6), turned to 0 degrees
- moved R8 3.84 mm to (114.4, 77.3)
- moved SW7 1.06 mm to (113.9, 76.6), turned to 180 degrees
- moved U0 0.82 mm to (114.4, 66.7)
- moved R4 0.78 mm to (118.2, 77.3)
- moved SW0 0.63 mm to (142.4, 64.9)
- moved SW4 0.32 mm to (139.3, 76.6)
Routing:
- net GND: track 61.9 -> 113.5 mm
- net Net-(R0-Pad2): track 5.06 -> 52.9 mm, vias 0 -> 1
- net +3V3: track 69.7 -> 104.0 mm, vias 2 -> 1
- net Net-(S0-Pad13C): track 22.9 -> 52.5 mm, vias 1 -> 0
- net Net-(SW4-Pad2): track 39.6 -> 54.6 mm
- net Net-(J0-Pad2): track 0.00 -> 12.1 mm, vias 0 -> 1
- net Net-(J0-Pad3): track 0.00 -> 10.5 mm, vias 0 -> 1
- net Net-(C0-Pad1): track 38.7 -> 48.9 mm
- net Net-(R7-Pad2): track 6.98 -> 16.3 mm
- net Net-(S0-Pad12): track 41.6 -> 46.1 mm
- net Net-(R4-Pad2): track 19.6 -> 23.3 mm
- net Net-(S0-Pad8C): track 21.8 -> 24.5 mm
- net (no net): track 2.28 -> 0.00 mm
- net Net-(S0-Pad7): track 15.6 -> 17.3 mm
- net Net-(S0-Pad11): track 35.0 -> 36.6 mm
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Other:
- board outline added: 38.1 x 21.6 mm

Commit message: PCB ready.
Parts:
- added G***: LOGO, kicad_bart:logo, F.Cu at (136.4, 62.9)
- J0: footprint Pin_Headers:Pin_Header_Straight_1x04 -> kicad_bart:SWD_PROGRAMMING_HEADER
- U0: footprint Housings_QFP:TQFP-32_7x7mm_Pitch0.8mm -> kicad_bart:TQFP-32_7x7mm_Pitch0.8mm
- renumbered SW4 to BTN4, SW7 to BTN7
Other:
- board text added: "2017"
- board text added: "EVPASCB1A (Panasonic 2.2N)"
- board text added: "LEFT"
- board text added: "LTP-305"
- board text added: "RIGHT"
- board text added: "STM32L031K6 (Cortex-M0+)"
